File: hardware/SplitX_2/SplitX_2.kicad_pcb (KiCad board)
At the start: 2 copper layers, 62.5 x 38 mm, 13 parts, among them J1 Screw_Terminal_01x02, J10 Screw_Terminal_01x02, J2 Screw_Terminal_01x03, J3 Screw_Terminal_01x03, J4 Screw_Terminal_01x03, J5 Screw_Terminal_01x03, J6 Screw_Terminal_01x03, J7 Screw_Terminal_01x03, J8 Screw_Terminal_01x03, J9 Screw_Terminal_01x03

Commit message: organized this folder and added a picture
Parts:
- removed G***: LOGO, custom_kicad_lib_sk:Train-Science logo small
- added REF**: OSHW-Logo2_9.8x8mm_SilkScreen, Symbol:OSHW-Logo2_9.8x8mm_SilkScreen, F.Cu at (223.4, 55.4)
- added REF**: OSHW-Logo2_9.8x8mm_SilkScreen, Symbol:OSHW-Logo2_9.8x8mm_SilkScreen, B.Cu at (223.4, 55.4)
