File: hardware/splitX_decoder/splitX_decoder.kicad_pcb (KiCad board)
At the start: 2 copper layers, 31.5 x 36 mm, 8 parts, among them J101 FEMALE, J102 FEMALE, J103 MALE, J104 MALE

Commit message: organized this folder and added a picture
Parts:
- removed G***: LOGO, custom_kicad_lib_sk:Train-Science logo small
- added REF**: OSHW-Logo_7.5x8mm_SilkScreen, Symbol:OSHW-Logo_7.5x8mm_SilkScreen, F.Cu at (165.2, 118.2)
