File: hardware/splitX_pluggable_8p/splitX_pluggable_8p.kicad_pcb (KiCad board)
At the start: 2 copper layers, 51.5 x 52 mm, 13 parts, among them J11 MALE, J12 MALE, J21 FEMALE, J22 FEMALE, J31 FEMALE, J32 FEMALE, J41 FEMALE, J42 FEMALE

Commit message: organized this folder and added a picture
Parts:
- removed G***: LOGO, custom_kicad_lib_sk:Train-Science logo small
